Commit message: Add two more robot models. They ugly :(

File: src/mpnp_simulation/models/kuka-omnirob-lwrs/model.urdf (robot description, URDF)
Before this commit: robot kuka-omnirob, 25 links, 24 joints
Links:
- link base_link: geometry collision box size=0.915855 0.547 0.585000; visual mesh filename=../kuka-omnirob/meshes/omnirobBaseRot.dae scale=1 1 1
- link bl_laser_link: geometry collision mesh filename=../kuka-omnirob/meshes/hokuyo.dae scale=1 1 1; visual mesh filename=../kuka-omnirob/meshes/hokuyo.dae scale=1 1 1
- link bl_wheel: geometry collision cylinder length=0.005 radius=0.125; visual mesh filename=../kuka-omnirob/meshes/omnirobBLWheelRot.dae scale=1 1 1
- link br_wheel: geometry collision cylinder length=0.005 radius=0.125; visual mesh filename=../kuka-omnirob/meshes/omnirobBRWheelRot.dae scale=1 1 1
- link fl_wheel: geometry collision cylinder length=0.005 radius=0.125; visual mesh filename=../kuka-omnirob/meshes/omnirobFLWheelRot.dae scale=1 1 1
- link fr_laser_link: geometry collision mesh filename=../kuka-omnirob/meshes/hokuyo.dae scale=1 1 1; visual mesh filename=../kuka-omnirob/meshes/hokuyo.dae scale=1 1 1
- link fr_wheel: geometry collision cylinder length=0.005 radius=0.125; visual mesh filename=../kuka-omnirob/meshes/omnirobFRWheelRot.dae scale=1 1 1
- link left_lwr_arm_1_link: geometry collision mesh filename=../kuka-lwr-4plus/meshes/convex/arm_segment_a_convex.stl scale=1.0 1.0 1.0; visual mesh filename=../kuka-lwr-4plus/meshes/arm_segment_a.dae scale=100 100 100
- link left_lwr_arm_2_link: geometry collision mesh filename=../kuka-lwr-4plus/meshes/convex/arm_segment_b_convex.stl scale=1.0 1.0 1.0; visual mesh filename=../kuka-lwr-4plus/meshes/arm_segment_b.dae scale=100 100 100
- link left_lwr_arm_3_link: geometry collision mesh filename=../kuka-lwr-4plus/meshes/convex/arm_segment_a_convex.stl scale=1.0 1.0 1.0; visual mesh filename=../kuka-lwr-4plus/meshes/arm_segment_a.dae scale=100 100 100
- link left_lwr_arm_4_link: geometry collision mesh filename=../kuka-lwr-4plus/meshes/convex/arm_segment_b_convex.stl scale=1.0 1.0 1.0; visual mesh filename=../kuka-lwr-4plus/meshes/arm_segment_b.dae scale=100 100 100
- link left_lwr_arm_5_link: geometry collision mesh filename=../kuka-lwr-4plus/meshes/convex/arm_segment_last_convex.stl scale=1.0 1.0 1.0; visual mesh filename=../kuka-lwr-4plus/meshes/arm_segment_last.dae scale=100 100 100
- link left_lwr_arm_6_link: geometry collision mesh filename=../kuka-lwr-4plus/meshes/convex/arm_wrist_convex.stl scale=1.0 1.0 1.0; visual mesh filename=../kuka-lwr-4plus/meshes/arm_wrist.dae scale=100 100 100
- link left_lwr_arm_7_link: geometry collision mesh filename=../kuka-lwr-4plus/meshes/arm_flanche.dae scale=100 100 100; visual mesh filename=../kuka-lwr-4plus/meshes/arm_flanche.dae scale=100 100 100
- link left_lwr_arm_base_link: geometry collision mesh filename=../kuka-lwr-4plus/meshes/convex/arm_base_convex.stl scale=0.9 0.9 0.9; visual mesh filename=../kuka-lwr-4plus/meshes/arm_base.dae scale=100 100 100
- link left_lwr_tool_link: geometry collision mesh filename=../kuka-lwr-4plus-triangle/TriangleFoot.stl scale=0.01 0.01 0.01; visual mesh filename=../kuka-lwr-4plus-triangle/TriangleFoot.stl scale=0.01 0.01 0.01
- link right_lwr_arm_1_link: geometry collision mesh filename=../kuka-lwr-4plus/meshes/convex/arm_segment_a_convex.stl scale=1.0 1.0 1.0; visual mesh filename=../kuka-lwr-4plus/meshes/arm_segment_a.dae scale=100 100 100
- link right_lwr_arm_2_link: geometry collision mesh filename=../kuka-lwr-4plus/meshes/convex/arm_segment_b_convex.stl scale=1.0 1.0 1.0; visual mesh filename=../kuka-lwr-4plus/meshes/arm_segment_b.dae scale=100 100 100
- link right_lwr_arm_3_link: geometry collision mesh filename=../kuka-lwr-4plus/meshes/convex/arm_segment_a_convex.stl scale=1.0 1.0 1.0; visual mesh filename=../kuka-lwr-4plus/meshes/arm_segment_a.dae scale=100 100 100
- link right_lwr_arm_4_link: geometry collision mesh filename=../kuka-lwr-4plus/meshes/convex/arm_segment_b_convex.stl scale=1.0 1.0 1.0; visual mesh filename=../kuka-lwr-4plus/meshes/arm_segment_b.dae scale=100 100 100
- link right_lwr_arm_5_link: geometry collision mesh filename=../kuka-lwr-4plus/meshes/convex/arm_segment_last_convex.stl scale=1.0 1.0 1.0; visual mesh filename=../kuka-lwr-4plus/meshes/arm_segment_last.dae scale=100 100 100
- link right_lwr_arm_6_link: geometry collision mesh filename=../kuka-lwr-4plus/meshes/convex/arm_wrist_convex.stl scale=1.0 1.0 1.0; visual mesh filename=../kuka-lwr-4plus/meshes/arm_wrist.dae scale=100 100 100
- link right_lwr_arm_7_link: geometry collision mesh filename=../kuka-lwr-4plus/meshes/arm_flanche.dae scale=100 100 100; visual mesh filename=../kuka-lwr-4plus/meshes/arm_flanche.dae scale=100 100 100
- link right_lwr_arm_base_link: geometry collision mesh filename=../kuka-lwr-4plus/meshes/convex/arm_base_convex.stl scale=0.9 0.9 0.9; visual mesh filename=../kuka-lwr-4plus/meshes/arm_base.dae scale=100 100 100
- link right_lwr_tool_link: geometry collision mesh filename=../kuka-lwr-4plus-triangle/TriangleFoot.stl scale=0.01 0.01 0.01; visual mesh filename=../kuka-lwr-4plus-triangle/TriangleFoot.stl scale=0.01 0.01 0.01

File: src/mpnp_simulation/models/kuka-omnirob/model.urdf (robot description, URDF)
Before this commit: robot kuka-omnirob, 7 links, 6 joints
Links:
- link base_link: geometry collision box size=0.915855 0.547 0.585000; visual mesh filename=kuka-omnirob/meshes/omnirobBaseRot.dae scale=1 1 1
- link bl_laser_link: geometry collision mesh filename=kuka-omnirob/meshes/hokuyo.dae scale=1 1 1; visual mesh filename=kuka-omnirob/meshes/hokuyo.dae scale=1 1 1
- link bl_wheel: geometry collision cylinder length=0.005 radius=0.125; visual mesh filename=kuka-omnirob/meshes/omnirobBLWheelRot.dae scale=1 1 1
- link br_wheel: geometry collision cylinder length=0.005 radius=0.125; visual mesh filename=kuka-omnirob/meshes/omnirobBRWheelRot.dae scale=1 1 1
- link fl_wheel: geometry collision cylinder length=0.005 radius=0.125; visual mesh filename=kuka-omnirob/meshes/omnirobFLWheelRot.dae scale=1 1 1
- link fr_laser_link: geometry collision mesh filename=kuka-omnirob/meshes/hokuyo.dae scale=1 1 1; visual mesh filename=kuka-omnirob/meshes/hokuyo.dae scale=1 1 1
- link fr_wheel: geometry collision cylinder length=0.005 radius=0.125; visual mesh filename=kuka-omnirob/meshes/omnirobFRWheelRot.dae scale=1 1 1
