Commit message: Connect the iisy arm to the mobile base and convert the urdf to sdf.

File: src/mpnp_simulation/models/kuka-omnirob-iisy/model.urdf (robot description, URDF)
Before this commit: robot kuka-omnirob, 7 links, 6 joints
Links:
- added link base
- added link flange
- added link link_1, mass 9.62E0; collision mesh filename=package://kuka_lbr_iisy_support/meshes/lbr_iisy15_r930/coll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; visual mesh filename=package://kuka_lbr_iisy_support/meshes/lbr_iisy15_r930/visu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
- added link link_2, mass 8.079E0; collision mesh filename=package://kuka_lbr_iisy_support/meshes/lbr_iisy15_r930/coll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; visual mesh filename=package://kuka_lbr_iisy_support/meshes/lbr_iisy15_r930/visu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
- added link link_3, mass 7.6604E0; collision mesh filename=package://kuka_lbr_iisy_support/meshes/lbr_iisy15_r930/coll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; visual mesh filename=package://kuka_lbr_iisy_support/meshes/lbr_iisy15_r930/visu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
- added link link_4, mass 5.7014E0; collision mesh filename=package://kuka_lbr_iisy_support/meshes/lbr_iisy15_r930/coll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; visual mesh filename=package://kuka_lbr_iisy_support/meshes/lbr_iisy15_r930/visu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
- added link link_5, mass 2.382E0; collision mesh filename=package://kuka_lbr_iisy_support/meshes/lbr_iisy15_r930/coll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; visual mesh filename=package://kuka_lbr_iisy_support/meshes/lbr_iisy15_r930/visu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
- added link link_6, mass 1.509E0; collision mesh filename=package://kuka_lbr_iisy_support/meshes/lbr_iisy15_r930/coll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; visual mesh filename=package://kuka_lbr_iisy_support/meshes/lbr_iisy15_r930/visu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
- added link m_base_link, mass 8.666E0; collision mesh filename=package://kuka_lbr_iisy_support/meshes/lbr_iisy15_r930/coll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; visual mesh filename=package://kuka_lbr_iisy_support/meshes/lbr_iisy15_r930/visu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
- added link tool0
Joints:
- added joint joint_1: type revolute, parent m_base_link, child link_1, origin xyz=0.0 0.0 0.0 rpy=-3.141592653589793 0.0 -0.0, axis 0.0 0.0 1.0, limit lower=-3.2288591161895095E0 upper=3.2288591161895095E0 effort=398.011277 velocity=3.490656
- added joint joint_2: type revolute, parent link_1, child link_2, origin xyz=0.0 0.0 -0.3 rpy=1.5707963267948966 0.0 -0.0, axis 0.0 0.0 1.0, limit lower=-4.014257279586958E0 upper=8.726646259971648E-1 effort=286.529873 velocity=3.490656
- added joint joint_3: type revolute, parent link_2, child link_3, origin xyz=0.385 0.0 0.0 rpy=0.0 0.0 -1.5707963267948966, axis 0.0 0.0 1.0, limit lower=-2.6179938779914944E0 upper=2.6179938779914944E0 effort=137.666701 velocity=3.490656
- added joint joint_4: type revolute, parent link_3, child link_4, origin xyz=0.0 0.0 0.0 rpy=1.5707963267948966 0.0 -0.0, axis 0.0 0.0 1.0, limit lower=-3.141592653589793E0 upper=3.141592653589793E0 effort=63.574238 velocity=4.014255
- added joint joint_5: type revolute, parent link_4, child link_5, origin xyz=0.0 0.0 -0.367 rpy=-1.5707963267948966 0.0 -0.0, axis 0.0 0.0 1.0, limit lower=-1.9198621771937625E0 upper=1.9198621771937625E0 effort=58.580298 velocity=4.537856
- added joint joint_6: type revolute, parent link_5, child link_6, origin xyz=0.0 0.0 0.0 rpy=1.5707963267948966 0.0 -0.0, axis 0.0 0.0 1.0, limit lower=-3.839724354387525E0 upper=3.839724354387525E0 effort=15.927568 velocity=7.504909
- added joint link6-flange: type fixed, parent link_6, child flange, origin xyz=0.0 0.0 -0.178 rpy=0 1.5707963267948966 -0.0
- added joint link6-tool0: type fixed, parent link_6, child tool0, origin xyz=0.0 0.0 -0.178 rpy=0 3.141592653589793 -0.0
- added joint m_base_link-base: type fixed, parent m_base_link, child base, origin xyz=0 0 0 rpy=0 0 0
- added joint m_base_link_joint: type fixed, parent base_link, child m_base_link, origin xyz=-0.3 0 0.6 rpy=0 0 0

Commit message: Comment out unused gazebo plugins, add fixed virtual joint between arm and mobile base.

File: src/mpnp_simulation/models/kuka-omnirob-iisy/model.urdf (robot description, URDF)
Before this commit: robot kuka-omnirob-iisy, 14 links, 12 joints
Links:
- removed link bl_laser_link
- removed link fr_laser_link
- link base_link: geometry collision box size=0.915855 0.547 0.585000; visual mesh filename=package://mpnp_simulation/models/kuka-omnirob-iisy/meshes/o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 scale=1 1 1
- link bl_wheel: geometry collision cylinder length=0.005 radius=0.125; visual mesh filename=package://mpnp_simulation/models/kuka-omnirob-iisy/meshes/o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 scale=1 1 1
- link br_wheel: geometry collision cylinder length=0.005 radius=0.125; visual mesh filename=package://mpnp_simulation/models/kuka-omnirob-iisy/meshes/o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 scale=1 1 1
- link fl_wheel: geometry collision cylinder length=0.005 radius=0.125; visual mesh filename=package://mpnp_simulation/models/kuka-omnirob-iisy/meshes/o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 scale=1 1 1
- link fr_wheel: geometry collision cylinder length=0.005 radius=0.125; visual mesh filename=package://mpnp_simulation/models/kuka-omnirob-iisy/meshes/o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 scale=1 1 1
Joints:
- removed joint bl_laser_joint
- removed joint fr_laser_joint
- added joint fixed_base_joint: type fixed, parent base_link, child m_base_link, origin xyz=-0.2 0.0 0.65 rpy=0.0 0.0 3.14
- joint joint_1: origin xyz=0.0 0.0 0.0 rpy=-3.141592653589793 0.0 -0.0 -> xyz=0.0 0.0 0.0 rpy=-3.141592653589793 0.0 3.14
