Commit message: Update urdf, remove unneeded sections.

File: src/mpnp_simulation/models/kuka-omnirob-iisy/lbr_iisy15_r930.urdf (robot description, URDF)
Before this commit: robot lbr_iisy15_r930, 11 links, 10 joints
Links:
- removed link flange
- removed link tool0
- removed link world
Joints:
- removed joint link6-flange
- removed joint link6-tool0
- removed joint world-base_link

File: src/mpnp_simulation/models/kuka-omnirob-iisy/model.urdf (robot description, URDF)
Before this commit: robot kuka-omnirob-iisy, 17 links, 16 joints
Links:
- removed link base
- removed link flange
- removed link tool0
Joints:
- removed joint link6-flange
- removed joint link6-tool0
- removed joint m_base_link-base
- removed joint m_base_link_joint

Commit message: Rename arm base link to arm_base_link for clarity.

File: src/mpnp_simulation/models/kuka-omnirob-iisy/lbr_iisy15_r930.urdf (robot description, URDF)
Before this commit: robot lbr_iisy15_r930, 7 links, 6 joints
Links:
- removed link base_link
- added link arm_base_link, mass 8.666E0; collision mesh filename=package://kuka_lbr_iisy_support/meshes/lbr_iisy15_r930/coll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; visual mesh filename=package://kuka_lbr_iisy_support/meshes/lbr_iisy15_r930/visu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
Joints:
- joint joint_1: parent base_link -> arm_base_link
