Commit message: Define macro xacro files for the mobile base and arm, then an urdf.xacro file to combine them.

File: src/mpnp_simulation/models/kuka-omnirob-iisy/kuka-omnirob-iisy.urdf.xacro (robot description, xacro)
@@ -1,8 +1,6 @@
 <?xml version="1.0"?>
-<robot xmlns:xacro="http://www.ros.org/wiki/xacro" name="lbr_iisy15_r930">
-  <!-- Import iisy macro files  -->
-  <xacro:include filename="$(find kuka_lbr_iisy_support)/urdf/lbr_iisy15_r930_macro.xacro"/>
-  <xacro:include filename="$(find kuka_lbr_iisy_support)/urdf/lbr_iisy_ros2_control_macro.xacro"/>
-  <!-- Read additional arguments  -->
+<robot xmlns:xacro="http://www.ros.org/wiki/xacro" name="kuka-omnirob-iisy">
+  <xacro:include filename="$(find mpnp_simulation)/models/kuka-omnirob-iisy/omnirob_macro.xacro"/>
+  <xacro:include filename="$(find mpnp_simulation)/models/kuka-omnirob-iisy/lbr_iisy15_r930_macro.xacro"/>
   <xacro:arg name="driver_version" default="rsi_only"/>
   <xacro:arg name="mode" default="hardware"/>
@@ -22,7 +20,13 @@
   <xacro:arg name="pitch" default="0"/>
   <xacro:arg name="yaw" default="0"/>
-  <xacro:kuka_lbr_iisy_ros2_control name="$(arg prefix)lbr_iisy15_r930" driver_version="$(arg driver_version)" client_ip="$(arg client_ip)" client_port="$(arg client_port)" mxa_client_port="$(arg mxa_client_port)" controller_ip="$(arg controller_ip)" prefix="$(arg prefix)" mode="$(arg mode)" use_gpio="$(arg use_gpio)" roundtrip_time="$(arg roundtrip_time)" verify_robot_model="$(arg verify_robot_model)" qos_config_file="$(arg qos_config_file)"/>
-  <xacro:kuka_lbr_iisy15_r930_robot prefix="$(arg prefix)" package_name="kuka_lbr_iisy_support">
+  <xacro:omnirob/>
+  <xacro:kuka_lbr_iisy15_r930_robot prefix="arm_" package_name="kuka_lbr_iisy_support">
     <origin xyz="$(arg x) $(arg y) $(arg z)" rpy="$(arg roll) $(arg pitch) $(arg yaw)"/>
   </xacro:kuka_lbr_iisy15_r930_robot>
+  <!-- Assemble omnirob and lbr iisy15 r930 -->
+  <joint name="arm_mount" type="fixed">
+    <child link="arm_base_link"/>
+    <origin rpy="0.0 0.0 0.0" xyz="0.38 0.12 0.65"/>
+    <parent link="platform_base_link"/>
+  </joint>
 </robot>

File: src/mpnp_simulation/models/kuka-omnirob-iisy/lbr_iisy15_r930_macro.xacro (robot description, xacro)
@@ -5,5 +5,4 @@
   <xacro:macro name="kuka_lbr_iisy15_r930_robot" params="prefix *origin package_name">
     <!-- links - main serial chain -->
-    <link name="world"/>
     <link name="${prefix}base_link">
       <collision>
@@ -147,9 +146,4 @@
     </link>
     <!-- joints - main serial chain -->
-    <joint name="${prefix}world-base_link" type="fixed">
-      <parent link="world"/>
-      <child link="${prefix}base_link"/>
-      <xacro:insert_block name="origin"/>
-    </joint>
     <joint name="${prefix}joint_1" type="revolute">
       <axis xyz="0.0 0.0 1.0"/>
@@ -194,25 +188,4 @@
       <parent link="${prefix}link_5"/>
     </joint>
-    <!-- ROS-Industrial 'base' frame - equivalent of 'KUKA ROBROOT'-->
-    <link name="${prefix}base"/>
-    <joint name="${prefix}base_link-base" type="fixed">
-      <origin xyz="0 0 0" rpy="0 0 0"/>
-      <parent link="${prefix}base_link"/>
-      <child link="${prefix}base"/>
-    </joint>
-    <!-- ROS-Industrial 'flange' frame - attachment point for EEF models -->
-    <link name="${prefix}flange"/>
-    <joint name="${prefix}link6-flange" type="fixed">
-      <child link="${prefix}flange"/>
-      <origin rpy="0 ${pi/2} -0.0" xyz="0.0 0.0 -0.178"/>
-      <parent link="${prefix}link_6"/>
-    </joint>
-    <!-- ROS-Industrial 'tool0' frame - all-zeros tool frame -->
-    <link name="${prefix}tool0"/>
-    <joint name="${prefix}link6-tool0" type="fixed">
-      <child link="${prefix}tool0"/>
-      <origin rpy="0 ${pi} -0.0" xyz="0.0 0.0 -0.178"/>
-      <parent link="${prefix}link_6"/>
-    </joint>
   </xacro:macro>
 </robot>
