Commit message: Add flange to iisy so an EE can be installed.

File: src/mpnp_simulation/models/kuka-omnirob-iisy/lbr_iisy15_r930_macro.xacro (robot description, xacro)
@@ -145,4 +145,5 @@
       </visual>
     </link>
+    <link name="${prefix}flange"/>
     <!-- joints - main serial chain -->
     <joint name="${prefix}joint_1" type="revolute">
@@ -188,4 +189,9 @@
       <parent link="${prefix}link_5"/>
     </joint>
+    <joint name="${prefix}link6-flange" type="fixed">
+      <child link="${prefix}flange"/>
+      <origin rpy="0 ${pi/2} -0.0" xyz="0.0 0.0 -0.178"/>
+      <parent link="${prefix}link_6"/>
+    </joint>
   </xacro:macro>
 </robot>
