Commit message: Define proper launch file for omnirob description and fix cmakelists

File: src/omnirob_description/urdf/omnirob_macro.xacro (robot description, xacro)
@@ -4,5 +4,5 @@
 	<xacro:macro name="omnirob">
 		<!--static>true</static-->
-		<link name="platform_base_link">
+		<link name="base_link">
 			<inertial>
 				<mass value="250" />
@@ -13,5 +13,5 @@
 				<origin rpy="0 0 0" xyz="0 0 0" />
 				<geometry>
-					<mesh filename="package://mpnp_simulation/models/kuka-omnirob-iisy/meshes/omnirobBaseRot.dae" scale="1 1 1" />
+					<mesh filename="package://omnirob_description/meshes/omnirobBaseRot.dae" scale="1 1 1" />
 				</geometry>
 			</visual>
@@ -32,5 +32,5 @@
 				<origin rpy="0 0 0" xyz="0 0.037 0" />
 				<geometry>
-					<mesh filename="package://mpnp_simulation/models/kuka-omnirob-iisy/meshes/omnirobBLWheelRot.dae" scale="1 1 1" />
+					<mesh filename="package://omnirob_description/meshes/omnirobBLWheelRot.dae" scale="1 1 1" />
 				</geometry>
 			</visual>
@@ -70,5 +70,5 @@
 			<origin rpy="0 3.14159 0" xyz="-0.347000 0.242000 0.130000" />
 			<axis xyz="0 1 0" />
-			<parent link="platform_base_link" />
+			<parent link="base_link" />
 			<child link="bl_wheel" />
 		</joint>
@@ -82,5 +82,5 @@
 				<origin rpy="0 0 0" xyz="0 -0.0 0" />
 				<geometry>
-					<mesh filename="package://mpnp_simulation/models/kuka-omnirob-iisy/meshes/omnirobBRWheelRot.dae" scale="1 1 1" />
+					<mesh filename="package://omnirob_description/meshes/omnirobBRWheelRot.dae" scale="1 1 1" />
 				</geometry>
 			</visual>
@@ -120,5 +120,5 @@
 			<origin rpy="0 0 0" xyz="-0.347000 -0.242000 0.130000" />
 			<axis xyz="0 1 0" />
-			<parent link="platform_base_link" />
+			<parent link="base_link" />
 			<child link="br_wheel" />
 		</joint>
@@ -132,5 +132,5 @@
 				<origin rpy="0 0 0" xyz="0 -0.0 0" />
 				<geometry>
-					<mesh filename="package://mpnp_simulation/models/kuka-omnirob-iisy/meshes/omnirobFRWheelRot.dae" scale="1 1 1" />
+					<mesh filename="package://omnirob_description/meshes/omnirobFRWheelRot.dae" scale="1 1 1" />
 				</geometry>
 			</visual>
@@ -170,5 +170,5 @@
 			<origin rpy="0 0 0" xyz="0.347000 -0.242000 0.130000" />
 			<axis xyz="0 1 0" />
-			<parent link="platform_base_link" />
+			<parent link="base_link" />
 			<child link="fr_wheel" />
 		</joint>
@@ -182,5 +182,5 @@
 				<origin rpy="0 0 0" xyz="0 0.0 0" />
 				<geometry>
-					<mesh filename="package://mpnp_simulation/models/kuka-omnirob-iisy/meshes/omnirobFLWheelRot.dae" scale="1 1 1" />
+					<mesh filename="package://omnirob_description/meshes/omnirobFLWheelRot.dae" scale="1 1 1" />
 				</geometry>
 			</visual>
@@ -220,5 +220,5 @@
 			<origin rpy="0 0 0" xyz="0.347000 0.242000 0.130000" />
 			<axis xyz="0 1 0" />
-			<parent link="platform_base_link" />
+			<parent link="base_link" />
 			<child link="fl_wheel" />
 		</joint>
