Commit message: Renaming

File: src/omnirob_description/urdf/omnirob.urdf.xacro (robot description, xacro)
@@ -2,4 +2,4 @@
 <robot xmlns:xacro="http://www.ros.org/wiki/xacro" name="kuka-omnirob-iisy">
   <xacro:include filename="$(find omnirob_description)/urdf/omnirob_macro.xacro"/>
-  <xacro:omnirob/>
+  <xacro:omnirob prefix="omnirob" package_name="omnirob_description"/>
 </robot>

File: src/omnirob_description/urdf/omnirob_macro.xacro (robot description, xacro)
@@ -2,7 +2,7 @@
 <robot name="omnirob" xmlns:controller="http://playerstage.sourceforge.net/gazebo/xmlschema/#controller" xmlns:interface="http://playerstage.sourceforge.net/gazebo/xmlschema/#interface" xmlns:sensor="http://playerstage.sourceforge.net/gazebo/xmlschema/#sensor" xmlns:xacro="http://www.ros.org/wiki/xacro">
     <!-- Helper xacros -->
-	<xacro:macro name="omnirob">
+	<xacro:macro name="omnirob" params="prefix package_name">
 		<!--static>true</static-->
-		<link name="base_link">
+		<link name="${prefix}_base_link">
 			<inertial>
 				<mass value="250" />
@@ -13,5 +13,5 @@
 				<origin rpy="0 0 0" xyz="0 0 0" />
 				<geometry>
-					<mesh filename="package://omnirob_description/meshes/omnirobBaseRot.dae" scale="1 1 1" />
+					<mesh filename="package://${package_name}/meshes/omnirobBaseRot.dae" scale="1 1 1" />
 				</geometry>
 			</visual>
@@ -32,5 +32,5 @@
 				<origin rpy="0 0 0" xyz="0 0.037 0" />
 				<geometry>
-					<mesh filename="package://omnirob_description/meshes/omnirobBLWheelRot.dae" scale="1 1 1" />
+					<mesh filename="package://${package_name}/meshes/omnirobBLWheelRot.dae" scale="1 1 1" />
 				</geometry>
 			</visual>
@@ -70,5 +70,5 @@
 			<origin rpy="0 3.14159 0" xyz="-0.347000 0.242000 0.130000" />
 			<axis xyz="0 1 0" />
-			<parent link="base_link" />
+			<parent link="${prefix}_base_link" />
 			<child link="bl_wheel" />
 		</joint>
@@ -82,5 +82,5 @@
 				<origin rpy="0 0 0" xyz="0 -0.0 0" />
 				<geometry>
-					<mesh filename="package://omnirob_description/meshes/omnirobBRWheelRot.dae" scale="1 1 1" />
+					<mesh filename="package://${package_name}/meshes/omnirobBRWheelRot.dae" scale="1 1 1" />
 				</geometry>
 			</visual>
@@ -120,5 +120,5 @@
 			<origin rpy="0 0 0" xyz="-0.347000 -0.242000 0.130000" />
 			<axis xyz="0 1 0" />
-			<parent link="base_link" />
+			<parent link="${prefix}_base_link" />
 			<child link="br_wheel" />
 		</joint>
@@ -132,5 +132,5 @@
 				<origin rpy="0 0 0" xyz="0 -0.0 0" />
 				<geometry>
-					<mesh filename="package://omnirob_description/meshes/omnirobFRWheelRot.dae" scale="1 1 1" />
+					<mesh filename="package://${package_name}/meshes/omnirobFRWheelRot.dae" scale="1 1 1" />
 				</geometry>
 			</visual>
@@ -170,5 +170,5 @@
 			<origin rpy="0 0 0" xyz="0.347000 -0.242000 0.130000" />
 			<axis xyz="0 1 0" />
-			<parent link="base_link" />
+			<parent link="${prefix}_base_link" />
 			<child link="fr_wheel" />
 		</joint>
@@ -182,5 +182,5 @@
 				<origin rpy="0 0 0" xyz="0 0.0 0" />
 				<geometry>
-					<mesh filename="package://omnirob_description/meshes/omnirobFLWheelRot.dae" scale="1 1 1" />
+					<mesh filename="package://${package_name}/meshes/omnirobFLWheelRot.dae" scale="1 1 1" />
 				</geometry>
 			</visual>
@@ -220,5 +220,5 @@
 			<origin rpy="0 0 0" xyz="0.347000 0.242000 0.130000" />
 			<axis xyz="0 1 0" />
-			<parent link="base_link" />
+			<parent link="${prefix}_base_link" />
 			<child link="fl_wheel" />
 		</joint>

Commit message: Trying mecanum drive plugin in gazebo.

File: src/omnirob_description/urdf/omnirob.urdf.xacro (robot description, xacro)
@@ -2,6 +2,8 @@
 <robot xmlns:xacro="http://www.ros.org/wiki/xacro" name="kuka-omnirob-iisy">
   <xacro:include filename="$(find omnirob_description)/urdf/omnirob_macro.xacro"/>
+  <!-- Gazebo plugin-->
+  <xacro:include filename="$(find omnirob_description)/urdf/omnirob.gazebo" />
   <!-- Import omnirob urdf file -->
-  <xacro:omnirob prefix="omnirob" package_name="omnirob_description"/>
+  <xacro:omnirob prefix="platform" package_name="omnirob_description"/>
   <!-- Import control_xacro -->
   <!-- <xacro:include filename="$(find omnirob_description)/config/omnirob.ros2_control.xacro"/> -->

File: src/omnirob_description/urdf/omnirob_macro.xacro (robot description, xacro)
@@ -1,11 +1,16 @@
 <?xml version="1.0" ?>
-<robot name="omnirob" xmlns:controller="http://playerstage.sourceforge.net/gazebo/xmlschema/#controller" xmlns:interface="http://playerstage.sourceforge.net/gazebo/xmlschema/#interface" xmlns:sensor="http://playerstage.sourceforge.net/gazebo/xmlschema/#sensor" xmlns:xacro="http://www.ros.org/wiki/xacro">
+<robot name="omnirob" xmlns:xacro="http://www.ros.org/wiki/xacro" xmlns:gz="http://gazebosim.org/schema">
     <!-- Helper xacros -->
 	<xacro:macro name="omnirob" params="prefix package_name">
-		<!--static>true</static-->
+		<link name="base_footprint"/>
+		<joint name="base_footprint_joint" type="fixed">
+			<origin rpy="0 0 0" xyz="0 0 0" />
+			<parent link="base_footprint" />
+			<child link="${prefix}_base_link" />
+		</joint>
 		<link name="${prefix}_base_link">
 			<inertial>
 				<mass value="250" />
-				<origin rpy="0 .0 0" xyz="0 -0.00000 0.24" />
+				<origin rpy="0 0 0.1" xyz="0 -0.00000 0.24" />
 				<inertia ixx="25.77086" ixy="-0.0" ixz="-0.0" iyy="53.79704" iyz="-0.0" izz="58.79601" />
 			</inertial>
@@ -36,40 +41,16 @@
 			</visual>
 			<collision>
-				<origin rpy="1.5708 0 0" xyz="0 0 0" />
 				<geometry>
-					<cylinder length="0.005" radius="0.125"/>
+					<sphere radius="0.1"/>
 				</geometry>
-				<surface>
-					<friction>
-						<ode>
-							<mu>1.5</mu>
-							<mu2>0.1</mu2>
-							<fdir1>1 1 0</fdir1>
-							<slip1>0</slip1>
-							<slip2>0</slip2>
-						</ode>
-					</friction>
-					<bounce>
-						<restitution_coefficient>0</restitution_coefficient>
-						<threshold>0</threshold>
-					</bounce>
-					<contact>
-						<ode>
-							<soft_cfm>0</soft_cfm>
-							<soft_erp>0.200000</soft_erp>
-							<kp>10000000000000.000000</kp>
-							<kd>100000000000.000000</kd>
-							<min_depth>0</min_depth>
-						</ode>
-					</contact>
-				</surface>
-				<laser_retro>0</laser_retro>
 			</collision>
 		</link>
 		<joint name="bl_wheel_joint" type="continuous">
-			<origin rpy="0 3.14159 0" xyz="-0.347000 0.242000 0.130000" />
-			<axis xyz="0 1 0" />
+			<origin rpy="0 0 0" xyz="-0.347000 0.242000 0.130000" />
+			<axis xyz="0 0 1" />
 			<parent link="${prefix}_base_link" />
 			<child link="bl_wheel" />
+			<limit effort="10000" velocity="10"/>
+    		<dynamics damping="1.0" friction="1.0"/>
 		</joint>
 		<link name="br_wheel">
@@ -86,40 +67,16 @@
 			</visual>
 			<collision>
-				<origin rpy="1.5708 0 0" xyz="0 0 0" />
 				<geometry>
-					<cylinder length="0.005" radius="0.125"/>
+					<sphere radius="0.1"/>
 				</geometry>
-				<surface>
-					<friction>
-						<ode>
-							<mu>1.5</mu>
-							<mu2>0.1</mu2>
-							<fdir1>1 -1 0</fdir1>
-							<slip1>0</slip1>
-							<slip2>0</slip2>
-						</ode>
-					</friction>
-					<bounce>
-						<restitution_coefficient>0</restitution_coefficient>
-						<threshold>0</threshold>
-					</bounce>
-					<contact>
-						<ode>
-							<soft_cfm>0</soft_cfm>
-							<soft_erp>0.200000</soft_erp>
-							<kp>10000000000000.000000</kp>
-							<kd>100000000000.000000</kd>
-							<min_depth>0</min_depth>
-						</ode>
-					</contact>
-				</surface>
-				<laser_retro>0</laser_retro>
 			</collision>
 		</link>
 		<joint name="br_wheel_joint" type="continuous">
 			<origin rpy="0 0 0" xyz="-0.347000 -0.242000 0.130000" />
-			<axis xyz="0 1 0" />
+			<axis xyz="0 0 1" />
 			<parent link="${prefix}_base_link" />
 			<child link="br_wheel" />
+			<limit effort="10000" velocity="10"/>
+    		<dynamics damping="1.0" friction="1.0"/>
 		</joint>
 		<link name="fr_wheel">
@@ -136,40 +93,16 @@
 			</visual>
 			<collision>
-				<origin rpy="1.5708 0 0" xyz="0 0 0" />
 				<geometry>
-					<cylinder length="0.005" radius="0.125"/>
+					<sphere radius="0.1"/>
 				</geometry>
-				<surface>
-					<friction>
-						<ode>
-							<mu>1.5</mu>
-							<mu2>0.1</mu2>
-							<fdir1>1 1 0</fdir1>
-							<slip1>0</slip1>
-							<slip2>0</slip2>
-						</ode>
-					</friction>
-					<bounce>
-						<restitution_coefficient>0</restitution_coefficient>
-						<threshold>0</threshold>
-					</bounce>
-					<contact>
-						<ode>
-							<soft_cfm>0</soft_cfm>
-							<soft_erp>0.200000</soft_erp>
-							<kp>10000000000000.000000</kp>
-							<kd>100000000000.000000</kd>
-							<min_depth>0</min_depth>
-						</ode>
-					</contact>
-				</surface>
-				<laser_retro>0</laser_retro>
 			</collision>
 		</link>
 		<joint name="fr_wheel_joint" type="continuous">
 			<origin rpy="0 0 0" xyz="0.347000 -0.242000 0.130000" />
-			<axis xyz="0 1 0" />
+			<axis xyz="0 0 1" />
 			<parent link="${prefix}_base_link" />
 			<child link="fr_wheel" />
+			<limit effort="10000" velocity="10"/>
+    		<dynamics damping="1.0" friction="1.0"/>
 		</joint>
 		<link name="fl_wheel">
@@ -186,41 +119,74 @@
 			</visual>
 			<collision>
-				<origin rpy="1.5708 0 0" xyz="0 0 0" />
 				<geometry>
-					<cylinder length="0.005" radius="0.125"/>
+					<sphere radius="0.1"/>
 				</geometry>
-				<surface>
-					<friction>
-						<ode>
-							<mu>1.5</mu>
-							<mu2>0.1</mu2>
-							<fdir1>1 -1 0</fdir1>
-							<slip1>0</slip1>
-							<slip2>0</slip2>
-						</ode>
-					</friction>
-					<bounce>
-						<restitution_coefficient>0</restitution_coefficient>
-						<threshold>0</threshold>
-					</bounce>
-					<contact>
-						<ode>
-							<soft_cfm>0</soft_cfm>
-							<soft_erp>0.200000</soft_erp>
-							<kp>10000000000000.000000</kp>
-							<kd>100000000000.000000</kd>
-							<min_depth>0</min_depth>
-						</ode>
-					</contact>
-				</surface>
-				<laser_retro>0</laser_retro>
 			</collision>
 		</link>
 		<joint name="fl_wheel_joint" type="continuous">
 			<origin rpy="0 0 0" xyz="0.347000 0.242000 0.130000" />
-			<axis xyz="0 1 0" />
+			<axis xyz="0 0 1" />
 			<parent link="${prefix}_base_link" />
 			<child link="fl_wheel" />
+			<limit effort="10000" velocity="10"/>
+    		<dynamics damping="1.0" friction="1.0"/>
 		</joint>
+		<!-- Gazebo frictions -->
+		<gazebo reference='fl_wheel'>
+			<collision>
+			<surface>
+				<friction>
+				<ode>
+					<mu>1.5</mu>
+					<mu2>0.0</mu2>
+					<fdir1 gz:expressed_in="base_footprint">1 -1 0</fdir1>
+				</ode>
+				</friction>
+			</surface>
+			</collision>
+		</gazebo>
+		<gazebo reference='bl_wheel'>
+			<collision>
+			<surface>
+				<friction>
+				<ode>
+					<mu>1.5</mu>
+					<mu2>0.0</mu2>
+					<fdir1 gz:expressed_in="base_footprint">1 1 0</fdir1>
+				</ode>
+				</friction>
+			</surface>
+			</collision>
+		</gazebo>
+		<gazebo reference='fr_wheel'>
+			<collision>
+			<surface>
+				<friction>
+				<ode>
+					<mu>1.5</mu>
+					<mu2>0.0</mu2>
+					<fdir1 gz:expressed_in="base_footprint">1 1 0</fdir1>
+				</ode>
+				</friction>
+			</surface>
+			</collision>
+		</gazebo>
+		<gazebo reference='br_wheel'>
+			<collision>
+			<surface>
+				<friction>
+				<ode>
+					<mu>1.5</mu>
+					<mu2>0.0</mu2>
+					<fdir1 gz:expressed_in="base_footprint">1 -1 0</fdir1>
+				</ode>
+				</friction>
+			</surface>
+			</collision>
+		</gazebo>
+		<gazebo reference="${prefix}_base_link">
+			<mu1>0.000002</mu1>
+			<mu2>0.000002</mu2>
+		</gazebo>
 	</xacro:macro>
 </robot>

Commit message: Fix mecanum wheels not working properly by just modeling them as spheres, and add proper gazebo friction parameters. It is omnidirectional now finally!

File: src/omnirob_description/urdf/omnirob.urdf.xacro (robot description, xacro)
@@ -2,10 +2,8 @@
 <robot xmlns:xacro="http://www.ros.org/wiki/xacro" name="kuka-omnirob-iisy">
   <xacro:include filename="$(find omnirob_description)/urdf/omnirob_macro.xacro"/>
-  <!-- Gazebo plugin-->
-  <xacro:include filename="$(find omnirob_description)/urdf/omnirob.gazebo" />
   <!-- Import omnirob urdf file -->
-  <xacro:omnirob prefix="platform" package_name="omnirob_description"/>
+  <xacro:omnirob prefix="platform_" package_name="omnirob_description"/>
   <!-- Import control_xacro -->
-  <!-- <xacro:include filename="$(find omnirob_description)/config/omnirob.ros2_control.xacro"/> -->
-  <!-- <xacro:omnirob_ros2_control/> -->
+  <xacro:include filename="$(find omnirob_description)/config/omnirob.ros2_control.xacro"/>
+  <xacro:omnirob_ros2_control/>
 </robot>

File: src/omnirob_description/urdf/omnirob_macro.xacro (robot description, xacro)
@@ -3,11 +3,5 @@
     <!-- Helper xacros -->
 	<xacro:macro name="omnirob" params="prefix package_name">
-		<link name="base_footprint"/>
-		<joint name="base_footprint_joint" type="fixed">
-			<origin rpy="0 0 0" xyz="0 0 0" />
-			<parent link="base_footprint" />
-			<child link="${prefix}_base_link" />
-		</joint>
-		<link name="${prefix}_base_link">
+		<link name="${prefix}base_link">
 			<inertial>
 				<mass value="250" />
@@ -48,6 +42,6 @@
 		<joint name="bl_wheel_joint" type="continuous">
 			<origin rpy="0 0 0" xyz="-0.347000 0.242000 0.130000" />
-			<axis xyz="0 0 1" />
-			<parent link="${prefix}_base_link" />
+			<axis xyz="0 1 0" />
+			<parent link="${prefix}base_link" />
 			<child link="bl_wheel" />
 			<limit effort="10000" velocity="10"/>
@@ -74,6 +68,6 @@
 		<joint name="br_wheel_joint" type="continuous">
 			<origin rpy="0 0 0" xyz="-0.347000 -0.242000 0.130000" />
-			<axis xyz="0 0 1" />
-			<parent link="${prefix}_base_link" />
+			<axis xyz="0 1 0" />
+			<parent link="${prefix}base_link" />
 			<child link="br_wheel" />
 			<limit effort="10000" velocity="10"/>
@@ -100,6 +94,6 @@
 		<joint name="fr_wheel_joint" type="continuous">
 			<origin rpy="0 0 0" xyz="0.347000 -0.242000 0.130000" />
-			<axis xyz="0 0 1" />
-			<parent link="${prefix}_base_link" />
+			<axis xyz="0 1 0" />
+			<parent link="${prefix}base_link" />
 			<child link="fr_wheel" />
 			<limit effort="10000" velocity="10"/>
@@ -126,6 +120,6 @@
 		<joint name="fl_wheel_joint" type="continuous">
 			<origin rpy="0 0 0" xyz="0.347000 0.242000 0.130000" />
-			<axis xyz="0 0 1" />
-			<parent link="${prefix}_base_link" />
+			<axis xyz="0 1 0" />
+			<parent link="${prefix}base_link" />
 			<child link="fl_wheel" />
 			<limit effort="10000" velocity="10"/>
@@ -140,5 +134,5 @@
 					<mu>1.5</mu>
 					<mu2>0.0</mu2>
-					<fdir1 gz:expressed_in="base_footprint">1 -1 0</fdir1>
+					<fdir1 gz:expressed_in="${prefix}base_link">1 -1 0</fdir1>
 				</ode>
 				</friction>
@@ -153,5 +147,5 @@
 					<mu>1.5</mu>
 					<mu2>0.0</mu2>
-					<fdir1 gz:expressed_in="base_footprint">1 1 0</fdir1>
+					<fdir1 gz:expressed_in="${prefix}base_link">1 1 0</fdir1>
 				</ode>
 				</friction>
@@ -166,5 +160,5 @@
 					<mu>1.5</mu>
 					<mu2>0.0</mu2>
-					<fdir1 gz:expressed_in="base_footprint">1 1 0</fdir1>
+					<fdir1 gz:expressed_in="${prefix}base_link">1 1 0</fdir1>
 				</ode>
 				</friction>
@@ -179,5 +173,5 @@
 					<mu>1.5</mu>
 					<mu2>0.0</mu2>
-					<fdir1 gz:expressed_in="base_footprint">1 -1 0</fdir1>
+					<fdir1 gz:expressed_in="${prefix}base_link">1 -1 0</fdir1>
 				</ode>
 				</friction>
@@ -185,5 +179,5 @@
 			</collision>
 		</gazebo>
-		<gazebo reference="${prefix}_base_link">
+		<gazebo reference="${prefix}base_link">
 			<mu1>0.000002</mu1>
 			<mu2>0.000002</mu2>
