Commit message: Build standalone kuka_iisy_description package.

File: src/kuka_iisy_description/urdf/lbr_iisy15_r930.urdf.xacro (robot description, xacro)
@@ -1,6 +1,5 @@
 <?xml version="1.0"?>
 <robot xmlns:xacro="http://www.ros.org/wiki/xacro" name="kuka-omnirob-iisy">
-  <xacro:include filename="$(find omnirob_description)/urdf/omnirob_macro.xacro"/>
-  <xacro:include filename="$(find mpnp_simulation)/models/kuka-omnirob-iisy/lbr_iisy15_r930_macro.xacro"/>
+  <xacro:include filename="$(find kuka_iisy_description)/urdf/lbr_iisy15_r930_macro.xacro"/>
   <xacro:arg name="driver_version" default="rsi_only"/>
   <xacro:arg name="mode" default="hardware"/>
@@ -20,12 +19,6 @@
   <xacro:arg name="pitch" default="0"/>
   <xacro:arg name="yaw" default="0"/>
-  <xacro:kuka_lbr_iisy15_r930_robot prefix="arm_" package_name="kuka_lbr_iisy_support">
+  <xacro:kuka_lbr_iisy15_r930_robot prefix="arm_" package_name="kuka_iisy_description">
     <origin xyz="$(arg x) $(arg y) $(arg z)" rpy="$(arg roll) $(arg pitch) $(arg yaw)"/>
   </xacro:kuka_lbr_iisy15_r930_robot>
-  <!-- Assemble lbr iisy15 r930 vgc10 vacuum gripper-->
-  <joint name="vg_mount" type="fixed">
-    <child link="arm_base_link"/>
-    <origin rpy="0.0 0.0 0.0" xyz="0.38 0.12 0.65"/>
-    <parent link="platform_base_link"/>
-  </joint>
 </robot>
