Commit message: Turn suction joints to prismatic so they don't all get clumped into one thing, and remove the virtual suction joint and link.

File: src/onrobot_vg_description/urdf/onrobot_vgc10_4cup.urdf.xacro (robot description, xacro)
@@ -2,4 +2,4 @@
 <robot name="onrobot_vgc10_model" xmlns:xacro="http://ros.org/wiki/xacro">
   <xacro:include filename="$(find onrobot_vg_description)/urdf/onrobot_vgc10_4cups_macro.xacro"/>
-  <xacro:onrobot_vgc10 prefix=""/>
+  <xacro:onrobot_vgc10/>
 </robot>

File: src/onrobot_vg_description/urdf/onrobot_vgc10_4cups_macro.xacro (robot description, xacro)
@@ -1,6 +1,6 @@
 <?xml version="1.0"?>
 <robot xmlns:xacro="http://ros.org/wiki/xacro">
-  <xacro:macro name="onrobot_vgc10" params="prefix">
-    <link name="${prefix}onrobot_vgc10_base_link">
+  <xacro:macro name="onrobot_vgc10">
+    <link name="onrobot_vgc10_base_link">
       <inertial>
         <origin xyz="0.0 0.0 0.0" rpy="0 0 0" />
@@ -24,49 +24,49 @@
       </collision>
     </link>
-    <link name="${prefix}suction1">
-      <inertial>
-        <origin xyz="0.0 0.0 0.0" rpy="0 0 0" />
-        <mass value="0.2" />
-        <inertia ixx="1.0E-03" ixy="1.0E-06" ixz="1.0E-06" iyy="1.0E-03" iyz="1.0E-06" izz="1.0E-03" />
-      </inertial>
-      <visual>
-        <origin xyz="0 0 0" rpy="0 0 0" />
-        <geometry>
-          <mesh filename="package://onrobot_vg_description/meshes/vgc10/visual/suction_cup_4cups.stl" />
-        </geometry>
-        <material name="">
-          <color rgba="0.9 0.9 0.9 1" />
-        </material>
-      </visual>
-      <collision>
-        <origin xyz="0 0 0" rpy="0 0 0" />
-        <geometry>
-          <mesh filename="package://onrobot_vg_description/meshes/vgc10/collision/suction_cup_4cups.stl" />
-        </geometry>
-      </collision>
-    </link>
-    <link name="${prefix}suction2">
-      <inertial>
-        <origin xyz="0.0 0.0 0.0" rpy="0 0 0" />
-        <mass value="0.2" />
-        <inertia ixx="1.0E-03" ixy="1.0E-06" ixz="1.0E-06" iyy="1.0E-03" iyz="1.0E-06" izz="1.0E-03" />
-      </inertial>
-      <visual>
-        <origin xyz="0 0 0" rpy="0 0 0" />
-        <geometry>
-          <mesh filename="package://onrobot_vg_description/meshes/vgc10/visual/suction_cup_4cups.stl" />
-        </geometry>
-        <material name="">
-          <color rgba="0.9 0.9 0.9 1" />
-        </material>
-      </visual>
-      <collision>
-        <origin xyz="0 0 0" rpy="0 0 0" />
-        <geometry>
-          <mesh filename="package://onrobot_vg_description/meshes/vgc10/collision/suction_cup_4cups.stl" />
-        </geometry>
-      </collision>
-    </link>
-    <link name="${prefix}suction3">
+    <link name="suction1">
+      <inertial>
+        <origin xyz="0.0 0.0 0.0" rpy="0 0 0" />
+        <mass value="0.2" />
+        <inertia ixx="1.0E-03" ixy="1.0E-06" ixz="1.0E-06" iyy="1.0E-03" iyz="1.0E-06" izz="1.0E-03" />
+      </inertial>
+      <visual>
+        <origin xyz="0 0 0" rpy="0 0 0" />
+        <geometry>
+          <mesh filename="package://onrobot_vg_description/meshes/vgc10/visual/suction_cup_4cups.stl" />
+        </geometry>
+        <material name="">
+          <color rgba="0.9 0.9 0.9 1" />
+        </material>
+      </visual>
+      <collision>
+        <origin xyz="0 0 0" rpy="0 0 0" />
+        <geometry>
+          <mesh filename="package://onrobot_vg_description/meshes/vgc10/collision/suction_cup_4cups.stl" />
+        </geometry>
+      </collision>
+    </link>
+    <link name="suction2">
+      <inertial>
+        <origin xyz="0.0 0.0 0.0" rpy="0 0 0" />
+        <mass value="0.2" />
+        <inertia ixx="1.0E-03" ixy="1.0E-06" ixz="1.0E-06" iyy="1.0E-03" iyz="1.0E-06" izz="1.0E-03" />
+      </inertial>
+      <visual>
+        <origin xyz="0 0 0" rpy="0 0 0" />
+        <geometry>
+          <mesh filename="package://onrobot_vg_description/meshes/vgc10/visual/suction_cup_4cups.stl" />
+        </geometry>
+        <material name="">
+          <color rgba="0.9 0.9 0.9 1" />
+        </material>
+      </visual>
+      <collision>
+        <origin xyz="0 0 0" rpy="0 0 0" />
+        <geometry>
+          <mesh filename="package://onrobot_vg_description/meshes/vgc10/collision/suction_cup_4cups.stl" />
+        </geometry>
+      </collision>
+    </link>
+    <link name="suction3">
       <inertial>
         <origin xyz="0.0 0.0 0.0" rpy="0 0 0" />
@@ -96,58 +96,65 @@
       </sensor>
     </link>
-    <link name="${prefix}suction4">
-      <inertial>
-        <origin xyz="0.0 0.0 0.0" rpy="0 0 0" />
-        <mass value="0.2" />
-        <inertia ixx="1.0E-03" ixy="1.0E-06" ixz="1.0E-06" iyy="1.0E-03" iyz="1.0E-06" izz="1.0E-03" />
-      </inertial>
-      <visual>
-        <origin xyz="0 0 0" rpy="0 0 0" />
-        <geometry>
-          <mesh filename="package://onrobot_vg_description/meshes/vgc10/visual/suction_cup_4cups.stl" />
-        </geometry>
-        <material name="">
-          <color rgba="0.9 0.9 0.9 1" />
-        </material>
-      </visual>
-      <collision>
-        <origin xyz="0 0 0" rpy="0 0 0" />
-        <geometry>
-          <mesh filename="package://onrobot_vg_description/meshes/vgc10/collision/suction_cup_4cups.stl" />
-        </geometry>
-      </collision>
-    </link>
-    <link name="${prefix}suction" />
-    <joint name="${prefix}suction_joint" type="fixed">
+    <link name="suction4">
+      <inertial>
+        <origin xyz="0.0 0.0 0.0" rpy="0 0 0" />
+        <mass value="0.2" />
+        <inertia ixx="1.0E-03" ixy="1.0E-06" ixz="1.0E-06" iyy="1.0E-03" iyz="1.0E-06" izz="1.0E-03" />
+      </inertial>
+      <visual>
+        <origin xyz="0 0 0" rpy="0 0 0" />
+        <geometry>
+          <mesh filename="package://onrobot_vg_description/meshes/vgc10/visual/suction_cup_4cups.stl" />
+        </geometry>
+        <material name="">
+          <color rgba="0.9 0.9 0.9 1" />
+        </material>
+      </visual>
+      <collision>
+        <origin xyz="0 0 0" rpy="0 0 0" />
+        <geometry>
+          <mesh filename="package://onrobot_vg_description/meshes/vgc10/collision/suction_cup_4cups.stl" />
+        </geometry>
+      </collision>
+    </link>
+    <!-- <link name="suction" /> -->
+    <!-- <joint name="suction_joint" type="prismatic">
       <origin xyz="0. 0. 0.08350" rpy="0 0 0" />
-      <parent link="${prefix}onrobot_vgc10_base_link" />
-      <child link="${prefix}suction" />
+      <parent link="onrobot_vgc10_base_link" />
+      <child link="suction" />
+      <axis xyz="0 0 1" />
+      <limit lower="0" upper="0.004" effort="10" velocity="0.01"/>
+    </joint> -->
+    <joint name="suction1_joint" type="prismatic">
+      <origin xyz="0.0175 0.0175 0.08350" rpy="0 0 0" />
+      <parent link="onrobot_vgc10_base_link" />
+      <child link="suction1" />
+      <axis xyz="0 0 1" />
+      <limit lower="0" upper="0.004" effort="10" velocity="0.01"/>
+    </joint>
+    <joint name="suction2_joint" type="prismatic">
+      <origin xyz="0.0175 -0.0175 0.08350" rpy="0 0 0" />
+      <parent link="onrobot_vgc10_base_link" />
+      <child link="suction2" />
+      <axis xyz="0 0 1" />
+      <limit lower="0" upper="0.004" effort="10" velocity="0.01"/>
+    </joint>
+    <joint name="suction3_joint" type="prismatic">
+      <origin xyz="-0.0175 0.0175 0.08350" rpy="0 0 0" />
+      <parent link="onrobot_vgc10_base_link" />
+      <child link="suction3" />
+      <axis xyz="0 0 1" />
+      <limit lower="0" upper="0.004" effort="10" velocity="0.01"/>
+    </joint>
+    <joint name="suction4_joint" type="prismatic">
+      <origin xyz="-0.0175 -0.0175 0.08350" rpy="0 0 0" />
+      <parent link="onrobot_vgc10_base_link" />
+      <child link="suction4" />
+      <axis xyz="0 0 1" />
+      <limit lower="0" upper="0.004" effort="10" velocity="0.01"/>
       <axis xyz="1 0 0" />
     </joint>
-    <joint name="${prefix}suction1_joint" type="fixed">
-      <origin xyz="0.0175 0.0175 0." rpy="0 0 0" />
-      <parent link="${prefix}suction" />
-      <child link="${prefix}suction1" />
-      <axis xyz="1 0 0" />
-    </joint>
-    <joint name="${prefix}suction2_joint" type="fixed">
-      <origin xyz="0.0175 -0.0175 0." rpy="0 0 0" />
-      <parent link="${prefix}suction" />
-      <child link="${prefix}suction2" />
-      <axis xyz="1 0 0" />
-    </joint>
-    <joint name="${prefix}suction3_joint" type="fixed">
-      <origin xyz="-0.0175 0.0175 0." rpy="0 0 0" />
-      <parent link="${prefix}suction" />
-      <child link="${prefix}suction3" />
-      <axis xyz="1 0 0" />
-    </joint>
-    <joint name="${prefix}suction4_joint" type="fixed">
-      <origin xyz="-0.0175 -0.0175 0." rpy="0 0 0" />
-      <parent link="${prefix}suction" />
-      <child link="${prefix}suction4" />
-      <axis xyz="1 0 0" />
-    </joint>
-    <gazebo reference="${prefix}suction1">
+    <gazebo reference="suction1">
+      <preserveFixedJoint>true</preserveFixedJoint>
       <sensor name='contact_sensor1' type='contact'>
         <update_rate>30</update_rate>
@@ -161,5 +168,6 @@
       </sensor>
     </gazebo>
-    <gazebo reference="${prefix}suction2">
+    <gazebo reference="suction2">
+      <preserveFixedJoint>true</preserveFixedJoint>
       <sensor name='contact_sensor2' type='contact'>
         <update_rate>30</update_rate>
@@ -173,5 +181,6 @@
       </sensor>
     </gazebo>
-    <gazebo reference="${prefix}suction3">
+    <gazebo reference="suction3">
+      <preserveFixedJoint>true</preserveFixedJoint>
       <sensor name='contact_sensor3' type='contact'>
         <update_rate>30</update_rate>
@@ -185,5 +194,6 @@
       </sensor>
     </gazebo>
-    <gazebo reference="${prefix}suction4">
+    <gazebo reference="suction4">
+      <preserveFixedJoint>true</preserveFixedJoint>
       <sensor name='contact_sensor4' type='contact'>
         <update_rate>30</update_rate>
@@ -196,4 +206,12 @@
         </plugin>
       </sensor>
+    </gazebo>
+    <gazebo>
+      <plugin filename="libVacuumToolPlugin.so" name="mpnp_plugins::VacuumToolPlugin">
+        <ros>
+          <namespace>/vacuum_tool/onrobot_vgc10</namespace>
+        </ros>
+        <tool_type>2</tool_type>
+      </plugin>
     </gazebo>
   </xacro:macro>
