Commit message: Update vacuum urdf to align with the plugin naming convention.

File: src/onrobot_vg_description/urdf/onrobot_vgc10_4cups_macro.xacro (robot description, xacro)
@@ -45,4 +45,16 @@
         </geometry>
       </collision>
+      <sensor name='contact_sensor' type='contact'>
+        <update_rate>30</update_rate>
+        <contact>
+          <collision>collision</collision>
+        </contact>
+        <plugin
+          filename="libContactPlugin.so"
+          name="mpnp_plugins::ContactPlugin">
+          <search_term>vg_4</search_term>
+          <update_rate>30</update_rate>
+        </plugin>
+      </sensor>
     </link>
     <link name="${prefix}suction2">
@@ -67,4 +79,16 @@
         </geometry>
       </collision>
+      <sensor name='contact_sensor' type='contact'>
+        <update_rate>30</update_rate>
+        <contact>
+          <collision>collision</collision>
+        </contact>
+        <plugin
+          filename="libContactPlugin.so"
+          name="mpnp_plugins::ContactPlugin">
+          <search_term>vg_4</search_term>
+          <update_rate>30</update_rate>
+        </plugin>
+      </sensor>
     </link>
     <link name="${prefix}suction3">
@@ -89,4 +113,16 @@
         </geometry>
       </collision>
+      <sensor name='contact_sensor' type='contact'>
+        <update_rate>30</update_rate>
+        <contact>
+          <collision>collision</collision>
+        </contact>
+        <plugin
+          filename="libContactPlugin.so"
+          name="mpnp_plugins::ContactPlugin">
+          <search_term>vg_4</search_term>
+          <update_rate>30</update_rate>
+        </plugin>
+      </sensor>
     </link>
     <link name="${prefix}suction4">
@@ -111,7 +147,19 @@
         </geometry>
       </collision>
+      <sensor name='contact_sensor' type='contact'>
+        <update_rate>30</update_rate>
+        <contact>
+          <collision>collision</collision>
+        </contact>
+        <plugin
+          filename="libContactPlugin.so"
+          name="mpnp_plugins::ContactPlugin">
+          <search_term>vg_4</search_term>
+          <update_rate>30</update_rate>
+        </plugin>
+      </sensor>
     </link>
     <link name="${prefix}suction" />
-    <joint name="${prefix}_suction_joint" type="fixed">
+    <joint name="${prefix}suction_joint" type="fixed">
       <origin xyz="0. 0. 0.08350" rpy="0 0 0" />
       <parent link="${prefix}onrobot_vgc10_base_link" />
@@ -119,5 +167,5 @@
       <axis xyz="1 0 0" />
     </joint>
-    <joint name="${prefix}_suction1_joint" type="fixed">
+    <joint name="${prefix}suction1_joint" type="fixed">
       <origin xyz="0.0175 0.0175 0." rpy="0 0 0" />
       <parent link="${prefix}suction" />
@@ -125,5 +173,5 @@
       <axis xyz="1 0 0" />
     </joint>
-    <joint name="${prefix}_suction2_joint" type="fixed">
+    <joint name="${prefix}suction2_joint" type="fixed">
       <origin xyz="0.0175 -0.0175 0." rpy="0 0 0" />
       <parent link="${prefix}suction" />
@@ -131,5 +179,5 @@
       <axis xyz="1 0 0" />
     </joint>
-    <joint name="${prefix}_suction3_joint" type="fixed">
+    <joint name="${prefix}suction3_joint" type="fixed">
       <origin xyz="-0.0175 0.0175 0." rpy="0 0 0" />
       <parent link="${prefix}suction" />
@@ -137,5 +185,5 @@
       <axis xyz="1 0 0" />
     </joint>
-    <joint name="${prefix}_suction4_joint" type="fixed">
+    <joint name="${prefix}suction4_joint" type="fixed">
       <origin xyz="-0.0175 -0.0175 0." rpy="0 0 0" />
       <parent link="${prefix}suction" />
@@ -143,4 +191,12 @@
       <axis xyz="1 0 0" />
     </joint>
+    <plugin
+      filename="libVacuumToolPlugin.so"
+      name="mpnp_plugins::VacuumToolPlugin">
+      <ros>
+        <namespace>/vacuum_tool/vgc10</namespace>
+      </ros>
+      <tool_type>2</tool_type>
+    </plugin>
   </xacro:macro>
 </robot>

Commit message: Make sdf file for the vacuum, need to redefine it properly. Update CMakeLists with new hooks and add gazebo plugins. Might not work this way, try sdf way instead since the plugins are gazebo system plugins.

File: src/onrobot_vg_description/urdf/onrobot_vgc10_4cups_macro.xacro (robot description, xacro)
@@ -45,4 +45,48 @@
         </geometry>
       </collision>
+    </link>
+    <link name="${prefix}suction2">
+      <inertial>
+        <origin xyz="0.0 0.0 0.0" rpy="0 0 0" />
+        <mass value="0.2" />
+        <inertia ixx="1.0E-03" ixy="1.0E-06" ixz="1.0E-06" iyy="1.0E-03" iyz="1.0E-06" izz="1.0E-03" />
+      </inertial>
+      <visual>
+        <origin xyz="0 0 0" rpy="0 0 0" />
+        <geometry>
+          <mesh filename="package://onrobot_vg_description/meshes/vgc10/visual/suction_cup_4cups.stl" />
+        </geometry>
+        <material name="">
+          <color rgba="0.9 0.9 0.9 1" />
+        </material>
+      </visual>
+      <collision>
+        <origin xyz="0 0 0" rpy="0 0 0" />
+        <geometry>
+          <mesh filename="package://onrobot_vg_description/meshes/vgc10/collision/suction_cup_4cups.stl" />
+        </geometry>
+      </collision>
+    </link>
+    <link name="${prefix}suction3">
+      <inertial>
+        <origin xyz="0.0 0.0 0.0" rpy="0 0 0" />
+        <mass value="0.2" />
+        <inertia ixx="1.0E-03" ixy="1.0E-06" ixz="1.0E-06" iyy="1.0E-03" iyz="1.0E-06" izz="1.0E-03" />
+      </inertial>
+      <visual>
+        <origin xyz="0 0 0" rpy="0 0 0" />
+        <geometry>
+          <mesh filename="package://onrobot_vg_description/meshes/vgc10/visual/suction_cup_4cups.stl" />
+        </geometry>
+        <material name="">
+          <color rgba="0.9 0.9 0.9 1" />
+        </material>
+      </visual>
+      <collision>
+        <origin xyz="0 0 0" rpy="0 0 0" />
+        <geometry>
+          <mesh filename="package://onrobot_vg_description/meshes/vgc10/collision/suction_cup_4cups.stl" />
+        </geometry>
+      </collision>
       <sensor name='contact_sensor' type='contact'>
         <update_rate>30</update_rate>
@@ -50,78 +94,4 @@
           <collision>collision</collision>
         </contact>
-        <plugin
-          filename="libContactPlugin.so"
-          name="mpnp_plugins::ContactPlugin">
-          <search_term>vg_4</search_term>
-          <update_rate>30</update_rate>
-        </plugin>
-      </sensor>
-    </link>
-    <link name="${prefix}suction2">
-      <inertial>
-        <origin xyz="0.0 0.0 0.0" rpy="0 0 0" />
-        <mass value="0.2" />
-        <inertia ixx="1.0E-03" ixy="1.0E-06" ixz="1.0E-06" iyy="1.0E-03" iyz="1.0E-06" izz="1.0E-03" />
-      </inertial>
-      <visual>
-        <origin xyz="0 0 0" rpy="0 0 0" />
-        <geometry>
-          <mesh filename="package://onrobot_vg_description/meshes/vgc10/visual/suction_cup_4cups.stl" />
-        </geometry>
-        <material name="">
-          <color rgba="0.9 0.9 0.9 1" />
-        </material>
-      </visual>
-      <collision>
-        <origin xyz="0 0 0" rpy="0 0 0" />
-        <geometry>
-          <mesh filename="package://onrobot_vg_description/meshes/vgc10/collision/suction_cup_4cups.stl" />
-        </geometry>
-      </collision>
-      <sensor name='contact_sensor' type='contact'>
-        <update_rate>30</update_rate>
-        <contact>
-          <collision>collision</collision>
-        </contact>
-        <plugin
-          filename="libContactPlugin.so"
-          name="mpnp_plugins::ContactPlugin">
-          <search_term>vg_4</search_term>
-          <update_rate>30</update_rate>
-        </plugin>
-      </sensor>
-    </link>
-    <link name="${prefix}suction3">
-      <inertial>
-        <origin xyz="0.0 0.0 0.0" rpy="0 0 0" />
-        <mass value="0.2" />
-        <inertia ixx="1.0E-03" ixy="1.0E-06" ixz="1.0E-06" iyy="1.0E-03" iyz="1.0E-06" izz="1.0E-03" />
-      </inertial>
-      <visual>
-        <origin xyz="0 0 0" rpy="0 0 0" />
-        <geometry>
-          <mesh filename="package://onrobot_vg_description/meshes/vgc10/visual/suction_cup_4cups.stl" />
-        </geometry>
-        <material name="">
-          <color rgba="0.9 0.9 0.9 1" />
-        </material>
-      </visual>
-      <collision>
-        <origin xyz="0 0 0" rpy="0 0 0" />
-        <geometry>
-          <mesh filename="package://onrobot_vg_description/meshes/vgc10/collision/suction_cup_4cups.stl" />
-        </geometry>
-      </collision>
-      <sensor name='contact_sensor' type='contact'>
-        <update_rate>30</update_rate>
-        <contact>
-          <collision>collision</collision>
-        </contact>
-        <plugin
-          filename="libContactPlugin.so"
-          name="mpnp_plugins::ContactPlugin">
-          <search_term>vg_4</search_term>
-          <update_rate>30</update_rate>
-        </plugin>
       </sensor>
     </link>
@@ -147,16 +117,4 @@
         </geometry>
       </collision>
-      <sensor name='contact_sensor' type='contact'>
-        <update_rate>30</update_rate>
-        <contact>
-          <collision>collision</collision>
-        </contact>
-        <plugin
-          filename="libContactPlugin.so"
-          name="mpnp_plugins::ContactPlugin">
-          <search_term>vg_4</search_term>
-          <update_rate>30</update_rate>
-        </plugin>
-      </sensor>
     </link>
     <link name="${prefix}suction" />
@@ -191,12 +149,52 @@
       <axis xyz="1 0 0" />
     </joint>
-    <plugin
-      filename="libVacuumToolPlugin.so"
-      name="mpnp_plugins::VacuumToolPlugin">
-      <ros>
-        <namespace>/vacuum_tool/vgc10</namespace>
-      </ros>
-      <tool_type>2</tool_type>
-    </plugin>
+    <gazebo reference="${prefix}suction1">
+      <sensor name='contact_sensor1' type='contact'>
+        <update_rate>30</update_rate>
+        <contact>
+          <collision>collision</collision>
+        </contact>
+        <plugin filename="libContactPlugin.so" name="mpnp_plugins::ContactPlugin">
+          <search_term>onrobot_vgc10</search_term>
+          <update_rate>30</update_rate>
+        </plugin>
+      </sensor>
+    </gazebo>
+    <gazebo reference="${prefix}suction2">
+      <sensor name='contact_sensor2' type='contact'>
+        <update_rate>30</update_rate>
+        <contact>
+          <collision>collision</collision>
+        </contact>
+        <plugin filename="libContactPlugin.so" name="mpnp_plugins::ContactPlugin">
+          <search_term>onrobot_vgc10</search_term>
+          <update_rate>30</update_rate>
+        </plugin>
+      </sensor>
+    </gazebo>
+    <gazebo reference="${prefix}suction3">
+      <sensor name='contact_sensor3' type='contact'>
+        <update_rate>30</update_rate>
+        <contact>
+          <collision>collision</collision>
+        </contact>
+        <plugin filename="libContactPlugin.so" name="mpnp_plugins::ContactPlugin">
+          <search_term>onrobot_vgc10</search_term>
+          <update_rate>30</update_rate>
+        </plugin>
+      </sensor>
+    </gazebo>
+    <gazebo reference="${prefix}suction4">
+      <sensor name='contact_sensor4' type='contact'>
+        <update_rate>30</update_rate>
+        <contact>
+          <collision>collision</collision>
+        </contact>
+        <plugin filename="libContactPlugin.so" name="mpnp_plugins::ContactPlugin">
+          <search_term>onrobot_vgc10</search_term>
+          <update_rate>30</update_rate>
+        </plugin>
+      </sensor>
+    </gazebo>
   </xacro:macro>
 </robot>

Commit message: Change suction joints to fixed, preserve these joints during conversion to sdf, update collision names and search term, and update the model.sdf for the gripper.

File: src/onrobot_vg_description/urdf/onrobot_vgc10_4cups_macro.xacro (robot description, xacro)
@@ -39,5 +39,5 @@
         </material>
       </visual>
-      <collision>
+      <collision name="suction1">
         <origin xyz="0 0 0" rpy="0 0 0" />
         <geometry>
@@ -61,5 +61,5 @@
         </material>
       </visual>
-      <collision>
+      <collision name="suction2">
         <origin xyz="0 0 0" rpy="0 0 0" />
         <geometry>
@@ -83,16 +83,10 @@
         </material>
       </visual>
-      <collision>
-        <origin xyz="0 0 0" rpy="0 0 0" />
-        <geometry>
-          <mesh filename="package://onrobot_vg_description/meshes/vgc10/collision/suction_cup_4cups.stl" />
-        </geometry>
-      </collision>
-      <sensor name='contact_sensor' type='contact'>
-        <update_rate>30</update_rate>
-        <contact>
-          <collision>collision</collision>
-        </contact>
-      </sensor>
+      <collision name="suction3">
+        <origin xyz="0 0 0" rpy="0 0 0" />
+        <geometry>
+          <mesh filename="package://onrobot_vg_description/meshes/vgc10/collision/suction_cup_4cups.stl" />
+        </geometry>
+      </collision>
     </link>
     <link name="suction4">
@@ -111,47 +105,34 @@
         </material>
       </visual>
-      <collision>
-        <origin xyz="0 0 0" rpy="0 0 0" />
-        <geometry>
-          <mesh filename="package://onrobot_vg_description/meshes/vgc10/collision/suction_cup_4cups.stl" />
-        </geometry>
-      </collision>
-    </link>
-    <!-- <link name="suction" /> -->
-    <!-- <joint name="suction_joint" type="prismatic">
-      <origin xyz="0. 0. 0.08350" rpy="0 0 0" />
-      <parent link="onrobot_vgc10_base_link" />
-      <child link="suction" />
-      <axis xyz="0 0 1" />
-      <limit lower="0" upper="0.004" effort="10" velocity="0.01"/>
-    </joint> -->
-    <joint name="suction1_joint" type="prismatic">
+      <collision name="suction4">
+        <origin xyz="0 0 0" rpy="0 0 0" />
+        <geometry>
+          <mesh filename="package://onrobot_vg_description/meshes/vgc10/collision/suction_cup_4cups.stl" />
+        </geometry>
+      </collision>
+    </link>
+    <joint name="suction1_joint" type="fixed">
       <origin xyz="0.0175 0.0175 0.08350" rpy="0 0 0" />
       <parent link="onrobot_vgc10_base_link" />
       <child link="suction1" />
       <axis xyz="0 0 1" />
-      <limit lower="0" upper="0.004" effort="10" velocity="0.01"/>
-    </joint>
-    <joint name="suction2_joint" type="prismatic">
+    </joint>
+    <joint name="suction2_joint" type="fixed">
       <origin xyz="0.0175 -0.0175 0.08350" rpy="0 0 0" />
       <parent link="onrobot_vgc10_base_link" />
       <child link="suction2" />
       <axis xyz="0 0 1" />
-      <limit lower="0" upper="0.004" effort="10" velocity="0.01"/>
-    </joint>
-    <joint name="suction3_joint" type="prismatic">
+    </joint>
+    <joint name="suction3_joint" type="fixed">
       <origin xyz="-0.0175 0.0175 0.08350" rpy="0 0 0" />
       <parent link="onrobot_vgc10_base_link" />
       <child link="suction3" />
       <axis xyz="0 0 1" />
-      <limit lower="0" upper="0.004" effort="10" velocity="0.01"/>
-    </joint>
-    <joint name="suction4_joint" type="prismatic">
+    </joint>
+    <joint name="suction4_joint" type="fixed">
       <origin xyz="-0.0175 -0.0175 0.08350" rpy="0 0 0" />
       <parent link="onrobot_vgc10_base_link" />
       <child link="suction4" />
       <axis xyz="0 0 1" />
-      <limit lower="0" upper="0.004" effort="10" velocity="0.01"/>
-      <axis xyz="1 0 0" />
     </joint>
     <gazebo reference="suction1">
@@ -159,8 +140,8 @@
         <update_rate>30</update_rate>
         <contact>
-          <collision>collision</collision>
-        </contact>
-        <plugin filename="libContactPlugin.so" name="mpnp_plugins::ContactPlugin">
-          <search_term>onrobot_vgc10</search_term>
+          <collision>suction1_collision</collision>
+        </contact>
+        <plugin filename="libContactPlugin.so" name="mpnp_plugins::ContactPlugin">
+          <search_term>vgc10</search_term>
           <update_rate>30</update_rate>
         </plugin>
@@ -171,8 +152,8 @@
         <update_rate>30</update_rate>
         <contact>
-          <collision>collision</collision>
-        </contact>
-        <plugin filename="libContactPlugin.so" name="mpnp_plugins::ContactPlugin">
-          <search_term>onrobot_vgc10</search_term>
+          <collision>suction2_collision</collision>
+        </contact>
+        <plugin filename="libContactPlugin.so" name="mpnp_plugins::ContactPlugin">
+          <search_term>vgc10</search_term>
           <update_rate>30</update_rate>
         </plugin>
@@ -183,8 +164,8 @@
         <update_rate>30</update_rate>
         <contact>
-          <collision>collision</collision>
-        </contact>
-        <plugin filename="libContactPlugin.so" name="mpnp_plugins::ContactPlugin">
-          <search_term>onrobot_vgc10</search_term>
+          <collision>suction3_collision</collision>
+        </contact>
+        <plugin filename="libContactPlugin.so" name="mpnp_plugins::ContactPlugin">
+          <search_term>vgc10</search_term>
           <update_rate>30</update_rate>
         </plugin>
@@ -195,8 +176,8 @@
         <update_rate>30</update_rate>
         <contact>
-          <collision>collision</collision>
-        </contact>
-        <plugin filename="libContactPlugin.so" name="mpnp_plugins::ContactPlugin">
-          <search_term>onrobot_vgc10</search_term>
+          <collision>suction4_collision</collision>
+        </contact>
+        <plugin filename="libContactPlugin.so" name="mpnp_plugins::ContactPlugin">
+          <search_term>vgc10</search_term>
           <update_rate>30</update_rate>
         </plugin>
@@ -211,4 +192,16 @@
       </plugin>
     </gazebo>
+    <gazebo reference="suction1_joint">
+      <preserveFixedJoint>true</preserveFixedJoint>
+    </gazebo>
+    <gazebo reference="suction2_joint">
+      <preserveFixedJoint>true</preserveFixedJoint>
+    </gazebo>
+    <gazebo reference="suction3_joint">
+      <preserveFixedJoint>true</preserveFixedJoint>
+    </gazebo>
+    <gazebo reference="suction4_joint">
+      <preserveFixedJoint>true</preserveFixedJoint>
+    </gazebo>
   </xacro:macro>
 </robot>
