Commit message: Fix launch files and parameters. Now everything works!

File: src/omnirob_iisy_vgc10_moveit_config/config/kuka_omnirob_iisy_vgc10.ros2_control.xacro (robot description, xacro)
@@ -50,6 +50,26 @@
                 <state_interface name="velocity"/>
             </joint>
+            <joint name="fl_wheel_joint">
+                <command_interface name="velocity"/>
+                <state_interface name="velocity"/>
+                <state_interface name="position"/>
+            </joint>
+            <joint name="fr_wheel_joint">
+                <command_interface name="velocity"/>
+                <state_interface name="velocity"/>
+                <state_interface name="position"/>
+            </joint>
+            <joint name="bl_wheel_joint">
+                <command_interface name="velocity"/>
+                <state_interface name="velocity"/>
+                <state_interface name="position"/>
+            </joint>
+            <joint name="br_wheel_joint">
+                <command_interface name="velocity"/>
+                <state_interface name="velocity"/>
+                <state_interface name="position"/>
+            </joint>
         </ros2_control>
-         <gazebo>
+        <gazebo>
             <plugin filename="gz_ros2_control-system" name="gz_ros2_control::GazeboSimROS2ControlPlugin">
                 <parameters>$(find omnirob_iisy_vgc10_moveit_config)/config/ros2_controllers.yaml</parameters>

File: src/omnirob_iisy_vgc10_moveit_config/config/kuka_omnirob_iisy_vgc10.urdf.xacro (robot description, xacro)
@@ -6,6 +6,6 @@
     <!-- Import control_xacro -->
     <xacro:include filename="kuka_omnirob_iisy_vgc10.ros2_control.xacro" />
-    <xacro:include filename="$(find omnirob_description)/config/omnirob.ros2_control.xacro"/>
+    <!-- <xacro:include filename="$(find omnirob_description)/config/omnirob.ros2_control.xacro" /> -->
     <xacro:kuka_omnirob_iisy_vgc10_ros2_control name="FakeSystem" initial_positions_file="$(arg initial_positions_file)"/>
-    <xacro:omnirob_ros2_control/>
+    <!-- <xacro:omnirob_ros2_control/> -->
 </robot>

Commit message: Include suction joints in the ros2 control xacro.

File: src/omnirob_iisy_vgc10_moveit_config/config/kuka_omnirob_iisy_vgc10.ros2_control.xacro (robot description, xacro)
@@ -70,4 +70,24 @@
                 <state_interface name="position"/>
             </joint>
+            <joint name="suction1_joint">
+                <command_interface name="position"/>
+                <state_interface name="position"/>
+                <state_interface name="velocity"/>
+            </joint>
+            <joint name="suction2_joint">
+                <command_interface name="position"/>
+                <state_interface name="position"/>
+                <state_interface name="velocity"/>
+            </joint>
+            <joint name="suction3_joint">
+                <command_interface name="position"/>
+                <state_interface name="position"/>
+                <state_interface name="velocity"/>
+            </joint>
+            <joint name="suction4_joint">
+                <command_interface name="position"/>
+                <state_interface name="position"/>
+                <state_interface name="velocity"/>
+            </joint>
         </ros2_control>
         <gazebo>

Commit message: Remove suction joints from moveit control yamls, they are now fixed and won't be controlled.

File: src/omnirob_iisy_vgc10_moveit_config/config/kuka_omnirob_iisy_vgc10.ros2_control.xacro (robot description, xacro)
@@ -70,24 +70,4 @@
                 <state_interface name="position"/>
             </joint>
-            <joint name="suction1_joint">
-                <command_interface name="position"/>
-                <state_interface name="position"/>
-                <state_interface name="velocity"/>
-            </joint>
-            <joint name="suction2_joint">
-                <command_interface name="position"/>
-                <state_interface name="position"/>
-                <state_interface name="velocity"/>
-            </joint>
-            <joint name="suction3_joint">
-                <command_interface name="position"/>
-                <state_interface name="position"/>
-                <state_interface name="velocity"/>
-            </joint>
-            <joint name="suction4_joint">
-                <command_interface name="position"/>
-                <state_interface name="position"/>
-                <state_interface name="velocity"/>
-            </joint>
         </ros2_control>
         <gazebo>
