Commit message: Add a suction join and link as eef, and turn on tf viz by default.

File: onrobot_vg_description/urdf/onrobot_vgc10_4cups_macro.xacro (robot description, xacro)
@@ -112,25 +112,44 @@
       </collision>
     </link>
+    <link name="suction">
+      <inertial>
+        <origin xyz="0.0 0.0 0.0" rpy="0 0 0" />
+        <mass value="0.2" />
+        <inertia ixx="1.0E-03" ixy="1.0E-06" ixz="1.0E-06" iyy="1.0E-03" iyz="1.0E-06" izz="1.0E-03" />
+      </inertial>
+      <collision name="suction5">
+        <origin xyz="0 0 0" rpy="0 0 0" />
+        <geometry>
+          <mesh filename="package://onrobot_vg_description/meshes/vgc10/collision/suction_cup_4cups.stl" />
+        </geometry>
+      </collision>
+    </link>
+    <joint name="suction_joint" type="fixed">
+      <origin xyz="0 0 0.08350" rpy="0 0 0" />
+      <parent link="onrobot_vgc10_base_link" />
+      <child link="suction" />
+      <axis xyz="0 0 1" />
+    </joint>
     <joint name="suction1_joint" type="fixed">
-      <origin xyz="0.0175 0.0175 0.08350" rpy="0 0 0" />
-      <parent link="onrobot_vgc10_base_link" />
+      <origin xyz="0.0175 0.0175 0.0" rpy="0 0 0" />
+      <parent link="suction" />
       <child link="suction1" />
       <axis xyz="0 0 1" />
     </joint>
     <joint name="suction2_joint" type="fixed">
-      <origin xyz="0.0175 -0.0175 0.08350" rpy="0 0 0" />
-      <parent link="onrobot_vgc10_base_link" />
+      <origin xyz="0.0175 -0.0175 0.0" rpy="0 0 0" />
+      <parent link="suction" />
       <child link="suction2" />
       <axis xyz="0 0 1" />
     </joint>
     <joint name="suction3_joint" type="fixed">
-      <origin xyz="-0.0175 0.0175 0.08350" rpy="0 0 0" />
-      <parent link="onrobot_vgc10_base_link" />
+      <origin xyz="-0.0175 0.0175 0.0" rpy="0 0 0" />
+      <parent link="suction" />
       <child link="suction3" />
       <axis xyz="0 0 1" />
     </joint>
     <joint name="suction4_joint" type="fixed">
-      <origin xyz="-0.0175 -0.0175 0.08350" rpy="0 0 0" />
-      <parent link="onrobot_vgc10_base_link" />
+      <origin xyz="-0.0175 -0.0175 0.0" rpy="0 0 0" />
+      <parent link="suction" />
       <child link="suction4" />
       <axis xyz="0 0 1" />
