Commit message: Remove arm y-offset and find decent position offset for base pathing.

File: mpnp_simulation/models/kuka_omnirob_iisy_vgc10.urdf.xacro (robot description, xacro)
@@ -37,5 +37,5 @@
   <joint name="arm_mount" type="fixed">
     <child link="arm_base_link"/>
-    <origin rpy="0.0 0.0 0.0" xyz="0.38 0.12 0.65"/>
+    <origin rpy="0.0 0.0 0.0" xyz="0.38 0.0 0.65"/>
     <parent link="platform_base_link"/>
   </joint>
